File: ReSeed.sch (KiCad schematic (older format))
At the start: 42 parts, among them CN1 EDGE_CONNECTOR, CN2 AUDIO_OUT, CN3 AUDIO_IN, CN4 DB9_MALE, Q1 BC549C, Q2 BC549C, SW1 SW_INT_EXT, U1 MOS_8580, U2 4520, U3 74LS245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

Commit message: Back side complete?
Parts:
- Q1, Q2: footprint Package_TO_SOT_THT:TO-92_Inline -> Package_TO_SOT_THT:TO-92_HandSolder
Changed lines of the file:
@@
 F 0 "Q1" H 11746 1366 50  0000 L CNN
 F 1 "BC549C" H 11746 1275 50  0000 L CNN
-F 2 "Package_TO_SOT_THT:TO-92_Inline" H 11755 1245 50  0001 L CIN
+F 2 "Package_TO_SOT_THT:TO-92_HandSolder" H 11755 1245 50  0001 L CIN
 F 3 "https://www.onsemi.com/pub/Collateral/BC550-D.pdf" H 11555 1320 50  0001 L CNN
 	1    11555 1320
@@
 F 0 "Q2" H 13606 1951 50  0000 L CNN
 F 1 "BC549C" H 13606 1860 50  0000 L CNN
-F 2 "Package_TO_SOT_THT:TO-92_Inline" H 13615 1830 50  0001 L CIN
+F 2 "Package_TO_SOT_THT:TO-92_HandSolder" H 13615 1830 50  0001 L CIN
 F 3 "https://www.onsemi.com/pub/Collateral/BC550-D.pdf" H 13415 1905 50  0001 L CNN
 	1    13415 1905

Commit message: Initial 1:1 replica complete
Parts:
- C4: footprint Capacitor_THT:CP_Radial_D6.3mm_P2.50mm -> Capacitor_THT:CP_Radial_D5.0mm_P2.00mm
Changed lines of the file:
@@
 F 0 "C4" V 12397 1625 50  0000 C CNN
 F 1 "10u" V 12306 1625 50  0000 C CNN
-F 2 "Capacitor_THT:CP_Radial_D6.3mm_P2.50mm" H 12145 1625 50  0001 C CNN
+F 2 "Capacitor_THT:CP_Radial_D5.0mm_P2.00mm" H 12145 1625 50  0001 C CNN
 F 3 "~" H 12145 1625 50  0001 C CNN
 	1    12145 1625

Commit message: Switch to radial inductor and make boards slightly shorter
Parts:
- removed CN2: AUDIO_OUT, Connector_Audio:Jack_3.5mm_Ledino_KB3SPRS_Horizontal, symbol Connector:AudioJack3
- removed CN3: AUDIO_IN, Connector_Audio:Jack_3.5mm_Ledino_KB3SPRS_Horizontal, symbol Connector:AudioJack3
- removed SW1: SW_INT_EXT, Connector_PinHeader_2.54mm:PinHeader_1x03_P2.54mm_Vertical, symbol Connector:Conn_01x03_Male
- added CN2: AUDIO_OUT, Connector_Audio:Jack_3.5mm_Ledino_KB3SPRS_Horizontal, symbol Connector:AudioJack3_SwitchTR
- added CN3: AUDIO_IN, Connector_Audio:Jack_3.5mm_Ledino_KB3SPRS_Horizontal, symbol Connector:AudioJack3_SwitchTR
- L1: footprint Inductor_THT:L_Axial_L7.0mm_D3.3mm_P12.70mm_Horizontal_Fastron_MICC -> Inductor_THT:L_Radial_D8.7mm_P5.00mm_Fastron_07HCP
Connections:
- wire segments 293 -> 294
- no-connect marks 24 -> 25
Changed lines of the file:
@@
 Sheet 1 1
 Title "ReSeed"
-Date "2022-02-09"
+Date "2022-02-12"
 Rev "1git"
 Comp "SukkoPera"
@@
 	1    0    0    -1
 $EndComp
-$Comp
-L Connector:AudioJack3 CN2
-U 1 1 62084245
-P 14965 1745
-F 0 "CN2" H 14685 1678 50  0000 R CNN
-F 1 "AUDIO_OUT" H 14685 1769 50  0000 R CNN
-F 2 "Connector_Audio:Jack_3.5mm_Ledino_KB3SPRS_Horizontal" H 14965 1745 50  0001 C CNN
-F 3 "~" H 14965 1745 50  0001 C CNN
-	1    14965 1745
-	-1   0    0    1
-$EndComp
-$Comp
-L Connector:AudioJack3 CN3
-U 1 1 6208459B
-P 14965 3115
-F 0 "CN3" H 14685 3048 50  0000 R CNN
-F 1 "AUDIO_IN" H 14685 3139 50  0000 R CNN
-F 2 "Connector_Audio:Jack_3.5mm_Ledino_KB3SPRS_Horizontal" H 14965 3115 50  0001 C CNN
-F 3 "~" H 14965 3115 50  0001 C CNN
-	1    14965 3115
-	-1   0    0    1
-$EndComp
 Wire Wire Line
 	1880 4725 1740 4725
@@
 F 0 "L1" H 6972 9216 50  0000 L CNN
 F 1 "680u" H 6972 9125 50  0000 L CNN
-F 2 "Inductor_THT:L_Axial_L7.0mm_D3.3mm_P12.70mm_Horizontal_Fastron_MICC" H 6920 9170 50  0001 C CNN
+F 2 "Inductor_THT:L_Radial_D8.7mm_P5.00mm_Fastron_07HCP" H 6920 9170 50  0001 C CNN
 F 3 "~" H 6920 9170 50  0001 C CNN
 	1    6920 9170
@@
 ~sid
 $Comp
-L Connector:Conn_01x03_Male SW1
-U 1 1 62FFCD54
-P 14415 2145
-F 0 "SW1" V 14395 2370 50  0000 R CNN
-F 1 "SW_INT_EXT" V 14305 2550 50  0000 R CNN
-F 2 "Connector_PinHeader_2.54mm:PinHeader_1x03_P2.54mm_Vertical" H 14415 2145 50  0001 C CNN
-F 3 "~" H 14415 2145 50  0001 C CNN
-	1    14415 2145
-	0    -1   -1   0
-$EndComp
-$Comp
 L Device:R R1
 U 1 1 63010374
@@
 Wire Wire Line
 	13515 1645 13895 1645
-Wire Wire Line
-	14765 1845 14650 1845
-Wire Wire Line
-	14650 1845 14650 2230
 $Comp
 L power:GND #PWR010
@@
 	1    0    0    -1
 $EndComp
-Wire Wire Line
-	14765 1645 14515 1645
 Text Label 1275 4625 0    50   ~ 0
 phi2
-Text Label 13880 1845 0    50   ~ 0
-ext_audio
-Wire Wire Line
-	14315 1945 14315 1845
-Wire Wire Line
-	14315 1845 13880 1845
-Wire Wire Line
-	14515 1945 14515 1745
-Connection ~ 14515 1745
-Wire Wire Line
-	14515 1745 14765 1745
-Wire Wire Line
-	14515 1745 14515 1645
-Wire Wire Line
-	14415 1645 14415 1945
-Wire Wire Line
-	14195 1645 14415 1645
-Wire Wire Line
-	14765 3215 14650 3215
-Wire Wire Line
-	14650 3215 14650 3600
 $Comp
 L power:GND #PWR018
@@
 	-1   0    0    1
 $EndComp
+Text Notes 2485 7635 0    50   ~ 0
+SPARE
+Wire Wire Line
+	14765 1945 14650 1945
+Wire Wire Line
+	14650 1945 14650 2230
+Wire Wire Line
+	14765 1845 14650 1845
+Wire Wire Line
+	14650 1845 14650 1645
+Wire Wire Line
+	14195 1645 14650 1645
+Wire Wire Line
+	14650 1645 14765 1645
+Connection ~ 14650 1645
+Wire Wire Line
+	14765 1545 14330 1545
+Text Label 14330 1545 0    50   ~ 0
+ext_audio
+$Comp
+L Connector:AudioJack3_SwitchTR CN2
+U 1 1 637FDCD2
+P 14965 1845
+F 0 "CN2" H 14685 1678 50  0000 R CNN
+F 1 "AUDIO_OUT" H 14685 1769 50  0000 R CNN
+F 2 "Connector_Audio:Jack_3.5mm_Ledino_KB3SPRS_Horizontal" H 14965 1845 50  0001 C CNN
+F 3 "~" H 14965 1845 50  0001 C CNN
+	1    14965 1845
+	-1   0    0    1
+$EndComp
+NoConn ~ 14765 1745
+$Comp
+L Connector:AudioJack3_SwitchTR CN3
+U 1 1 6393D5DC
+P 14965 3215
+F 0 "CN3" H 14685 3048 50  0000 R CNN
+F 1 "AUDIO_IN" H 14685 3139 50  0000 R CNN
+F 2 "Connector_Audio:Jack_3.5mm_Ledino_KB3SPRS_Horizontal" H 14965 3215 50  0001 C CNN
+F 3 "~" H 14965 3215 50  0001 C CNN
+	1    14965 3215
+	-1   0    0    1
+$EndComp
+Wire Wire Line
+	14765 3315 14650 3315
+Wire Wire Line
+	14650 3315 14650 3600
+Wire Wire Line
+	13515 3015 14520 3015
+Wire Wire Line
+	14650 3315 14650 3115
+Wire Wire Line
+	14650 2915 14765 2915
+Connection ~ 14650 3315
 Wire Wire Line
 	14765 3115 14650 3115
-Wire Wire Line
-	14650 3115 14650 3015
+Connection ~ 14650 3115
+Wire Wire Line
+	14650 3115 14650 2915
+Wire Wire Line
+	14765 3215 14520 3215
+Wire Wire Line
+	14520 3215 14520 3015
 Wire Bus Line
 	9365 5800 9365 6055
@@
 Wire Bus Line
 	3870 2725 3870 4225
-Wire Wire Line
-	14765 3015 14650 3015
-Wire Wire Line
-	14650 3015 13515 3015
-Connection ~ 14650 3015
-Text Notes 2485 7635 0    50   ~ 0
-SPARE
+Connection ~ 14520 3015
+Wire Wire Line
+	14520 3015 14765 3015
 $EndSCHEMATC

Commit message: Switch to ground plane and lots of improvements
Parts:
- U2: value 4520 -> CD4520BE; MouserPN (none) -> 595-CD74HCT4520E
Other:
- note added: "AUDIO IS OUTPUT TO EXT_AUDIO,\nUNLESS A JACK IS INSERTED"
- note added: "MMMMH, I'M NOT TOO CONVINCED\nABOUT THE VALUES HERE..."
- note added: "SOMEONE SAYS THIS INTRODUCES\nDISTORTION. SO MAYBE WE\nSHOULD REDUCE GAIN?"
- note added: "THIS MUST BE CHANGED\nTO +12V FOR MOS 6581\n(40mA MAX)"
- note added: "USE 470pF\nFOR 6851"
- note added: "WHAT HAPPENS IF YOU WRITE TO THE PORT?\nYOU CAN CREATE SHORT CIRCUITS!\nTODO: CONSIDER ADDING DIODES, CONNECTING\nPIN 1 TO VCC OR SWITCHING TO 74244"
- note added: "WITH NO JACK, AUDIO_IN GETS SHORTED\nTO GND IN ORDER TO AVOID NOISE"
Changed lines of the file:
@@
 P 5915 2220
 F 0 "U2" H 5915 2587 50  0000 C CNN
-F 1 "4520" H 5915 2496 50  0000 C CNN
+F 1 "CD4520BE" H 5915 2496 50  0000 C CNN
 F 2 "Package_DIP:DIP-16_W7.62mm_Socket_LongPads" H 5915 2220 50  0001 C CNN
 F 3 "http://www.intersil.com/content/dam/Intersil/documents/cd45/cd4518bms-20bms.pdf" H 5915 2220 50  0001 C CNN
+F 4 "595-CD74HCT4520E" H 5915 2220 50  0001 C CNN "MouserPN"
 	1    5915 2220
 	1    0    0    -1
@@
 P 2615 8190
 F 0 "U2" H 2615 8557 50  0000 C CNN
-F 1 "4520" H 2615 8466 50  0000 C CNN
+F 1 "CD4520BE" H 2615 8466 50  0000 C CNN
 F 2 "Package_DIP:DIP-16_W7.62mm_Socket_LongPads" H 2615 8190 50  0001 C CNN
 F 3 "http://www.intersil.com/content/dam/Intersil/documents/cd45/cd4518bms-20bms.pdf" H 2615 8190 50  0001 C CNN
+F 4 "595-CD74HCT4520E" H 2615 8190 50  0001 C CNN "MouserPN"
 	2    2615 8190
 	1    0    0    -1
@@
 P 2885 9770
 F 0 "U2" H 3115 9816 50  0000 L CNN
-F 1 "4520" H 3115 9725 50  0000 L CNN
+F 1 "CD4520BE" H 3115 9725 50  0000 L CNN
 F 2 "Package_DIP:DIP-16_W7.62mm_Socket_LongPads" H 2885 9770 50  0001 C CNN
 F 3 "http://www.intersil.com/content/dam/Intersil/documents/cd45/cd4518bms-20bms.pdf" H 2885 9770 50  0001 C CNN
+F 4 "595-CD74HCT4520E" H 2885 9770 50  0001 C CNN "MouserPN"
 	3    2885 9770
 	1    0    0    -1
@@
 Wire Wire Line
 	14520 3015 14765 3015
+Text Notes 12200 8065 0    50   ~ 0
+WHAT HAPPENS IF YOU WRITE TO THE PORT?\nYOU CAN CREATE SHORT CIRCUITS!\nTODO: CONSIDER ADDING DIODES, CONNECTING\nPIN 1 TO VCC OR SWITCHING TO 74244
+Text Notes 9785 9570 0    50   ~ 0
+MMMMH, I'M NOT TOO CONVINCED\nABOUT THE VALUES HERE...
+Text Notes 11815 1160 0    50   ~ 0
+SOMEONE SAYS THIS INTRODUCES\nDISTORTION. SO MAYBE WE\nSHOULD REDUCE GAIN?
+Text Notes 14490 1315 0    50   ~ 0
+AUDIO IS OUTPUT TO EXT_AUDIO,\nUNLESS A JACK IS INSERTED
+Text Notes 14475 2750 0    50   ~ 0
+WITH NO JACK, AUDIO_IN GETS SHORTED\nTO GND IN ORDER TO AVOID NOISE
+Text Notes 6425 1640 2    50   ~ 0
+USE 470pF\nFOR 6851
+Text Notes 9180 8520 0    50   ~ 0
+THIS MUST BE CHANGED\nTO +12V FOR MOS 6581\n(40mA MAX)
 $EndSCHEMATC

Commit message: Rework power circuit
Parts:
- added C17: 100u/16V, Capacitor_THT:CP_Radial_D6.3mm_P2.50mm, symbol Device:CP1
- added C18: 100n, Capacitor_THT:C_Disc_D7.0mm_W2.5mm_P5.00mm, symbol Device:C
- C1, C6: MouserPN (none) -> 810-FG28X7R1H223KNT0
- C10, C11, C12, C13, C14, C9: MouserPN (none) -> 810-FG28X7R1H104KNT0
- C15: MouserPN (none) -> 810-FG28C0G1H470JNT0
- C16: value 47u -> 1000u/25V; footprint Capacitor_THT:CP_Radial_D6.3mm_P2.50mm -> Capacitor_THT:CP_Radial_D10.0mm_P5.00mm; MouserPN (none) -> 710-860020475018
- C2: MouserPN (none) -> 810-FG28C0G1H102JNT6
- C4: MouserPN (none) -> 710-860010472002
- C5: footprint Capacitor_THT:CP_Radial_D6.3mm_P2.50mm -> Capacitor_THT:CP_Radial_D5.0mm_P2.00mm; MouserPN (none) -> 710-860020472004
- C7, C8: MouserPN (none) -> 810-FG28C0G1H392JNT6
- CN1: MouserPN (none) -> ---
- L1: value 680u -> 330u; MouserPN (none) -> 652-RLB0914-331KL
- R10: value 75k -> 7.87k 1%
- R11: value 10k -> 1.2k 1%
- R9: value 10 -> 1 1%/0.5W; MouserPN (none) -> 603-MF0207FRE52-1R
- U1: MouserPN (none) -> :)
- U3: MouserPN (none) -> 595-SN74HCT245N
- U4: MouserPN (none) -> 556-AF16V8B15PU
- U5: MouserPN (none) -> 595-TL497ACNE4
Connections:
- net +5V: now also C17.1, C18.1
- net GND: now also C17.2, C18.2
Other:
- note added: "ADDITIONAL DECOUPLING\nFOR IMPROVED STABILITY"
- note added: "STEP-UP VOLTAGE\nREGULATOR"
- note added: "THIS CIRCUIT CAN PRODUCE EITHER\n+9V (140mA MAX) OR +12V (100mA MAX)\nBY CHANGING R1 ONLY. USE +12V FOR\nMOS 6581 AND +9V FOR MOS 8580."
- note added: "USE 11K FOR\nMOS 6581"
- note added: "USE 470pF\nFOR 6581"
- note removed: "5V -> 9V STEP-UP\nREGULATOR"
- note removed: "MMMMH, I'M NOT TOO CONVINCED\nABOUT THE VALUES HERE..."
- note removed: "THIS MUST BE CHANGED\nTO +12V FOR MOS 6581\n(40mA MAX)"
- note removed: "USE 470pF\nFOR 6851"
- moved on the sheet: L1, R10, R11, R9

Commit message: Add logo and license
Parts:
- added V0: LOGO, ReSeed:Logo, symbol void:Void
- added V1: LICENSE, ReSeed:cc_by_nc_sa, symbol void:Void
Changed lines of the file:
@@
 Comment1 "Replica of Christian Schäffner (Solder)'s SID Card for the Commodore 16/+4"
 Comment2 "http://solder-synergy.de/plus4/hardware/index.html"
-Comment3 ""
+Comment3 "Licensed under CC BY-NC-SA 4.0"
 Comment4 ""
 $EndDescr
@@
 Wire Notes Line
 	5895 1950 5895 1175
+$Comp
+L void:Void V0
+U 1 1 64138BAD
+P 15465 9505
+F 0 "V0" H 15543 9551 50  0000 L CNN
+F 1 "LOGO" H 15543 9460 50  0000 L CNN
+F 2 "ReSeed:Logo" H 15465 9505 50  0001 C CNN
+F 3 "" H 15465 9505 50  0001 C CNN
+	1    15465 9505
+	1    0    0    -1
+$EndComp
+$Comp
+L void:Void V1
+U 1 1 64138E7F
+P 15465 9740
+F 0 "V1" H 15543 9786 50  0000 L CNN
+F 1 "LICENSE" H 15543 9695 50  0000 L CNN
+F 2 "ReSeed:cc_by_nc_sa" H 15465 9740 50  0001 C CNN
+F 3 "" H 15465 9740 50  0001 C CNN
+	1    15465 9740
+	1    0    0    -1
+$EndComp
 Wire Bus Line
 	9365 5800 9365 6055

Commit message: Work in progress
Parts:
- removed C5: 22u, Capacitor_THT:CP_Radial_D5.0mm_P2.00mm, symbol Device:CP1
- removed Q2: BC549C, Package_TO_SOT_THT:TO-92_HandSolder, symbol Transistor_BJT:BC549
- removed R4: 1.5k, Resistor_THT:R_Axial_DIN0207_L6.3mm_D2.5mm_P10.16mm_Horizontal, symbol Device:R
- added C5: 100n, Capacitor_THT:C_Disc_D7.0mm_W2.5mm_P5.00mm, symbol Device:C
- C3: value 470 -> 470p
- Q1: value BC549C -> 2SC1815
- R10: MouserPN (none) -> 71-CMF557K8700FHEK
- R11: MouserPN (none) -> 603-MF0207FTE52-1K2
- R2: value 390 -> 1k
- RN1: MouserPN (none) -> 652-4609X-1LF-4.7K
- renumbered R6 to R3, R3 to R4
Connections:
- net +5V: no longer R2.2
- net +9V: now also C5.2
- net GND: now also R2.1, C5.1
- net audio_in: now reaches C9.2, R7.2, U1.26 (AUDIO_IN)
- net audio_out: now reaches R1.2, U1.27 (AUDIO_OUT)
- net audio_out: now also R2.2
- net at RV1.2: now also CN2.R, CN2.T
Other:
- note added: "ANY VALUE BETWEEN\n1K-10K IS PROBABLY FINE"
- note added: "BC549C CAN BE USED TOO,\nWITH HIGHER NOISE THOUGH"
- note removed: "SOMEONE SAYS THIS INTRODUCES\nDISTORTION. SO MAYBE WE\nSHOULD REDUCE GAIN?"
- moved on the sheet: C2, C3, C4, Q1, R1, R3, RV1

Commit message: Almost there...
Parts:
- added RV2: 1M, ReSeed:Potentiometer_Vertical, symbol Device:R_POT
- added SW1: SW_DIGIFIX, Connector_PinHeader_2.54mm:PinHeader_1x03_P2.54mm_Vertical, symbol Connector:Conn_01x03_Male
- RV1: footprint Potentiometer_THT:Potentiometer_ACP_CA9-V10_Vertical_Hole -> ReSeed:Potentiometer_Vertical
Connections:
- net audio_in: now also SW1.2 (Pin_2); no longer R7.2
- new net: R7.2, RV2.2
- new net: RV2.1, SW1.3 (Pin_3)
- no-connect marks 25 -> 27
Other:
- moved on the sheet: R7
Changed lines of the file:
@@
 F 0 "RV1" H 13350 1951 50  0000 R CNN
 F 1 "10k" H 13350 1860 50  0000 R CNN
-F 2 "Potentiometer_THT:Potentiometer_ACP_CA9-V10_Vertical_Hole" H 13420 1905 50  0001 C CNN
+F 2 "ReSeed:Potentiometer_Vertical" H 13420 1905 50  0001 C CNN
 F 3 "~" H 13420 1905 50  0001 C CNN
 	1    13420 1905
@@
 Wire Wire Line
 	13515 3015 12685 3015
-Wire Wire Line
-	12385 3015 11655 3015
-Wire Wire Line
-	11655 3015 11655 3145
-Wire Wire Line
-	11655 3445 11655 3520
-$Comp
-L power:GND #PWR016
-U 1 1 6340CB1D
-P 11655 3520
-F 0 "#PWR016" H 11655 3270 50  0001 C CNN
-F 1 "GND" H 11660 3347 50  0000 C CNN
-F 2 "" H 11655 3520 50  0001 C CNN
-F 3 "" H 11655 3520 50  0001 C CNN
-	1    11655 3520
-	1    0    0    -1
-$EndComp
-Connection ~ 11655 3015
-Wire Wire Line
-	11655 3015 10400 3015
-$Comp
-L Device:R R7
-U 1 1 6340C3F1
-P 11655 3295
-F 0 "R7" H 11585 3249 50  0000 R CNN
-F 1 "180k" H 11585 3340 50  0000 R CNN
-F 2 "Resistor_THT:R_Axial_DIN0207_L6.3mm_D2.5mm_P10.16mm_Horizontal" V 11585 3295 50  0001 C CNN
-F 3 "~" H 11655 3295 50  0001 C CNN
-	1    11655 3295
-	-1   0    0    1
-$EndComp
 Text Notes 2485 7635 0    50   ~ 0
 SPARE
@@
 Wire Wire Line
 	13420 940  13420 1085
-Wire Bus Line
-	9365 5800 9365 6055
-Wire Bus Line
-	7120 2320 7120 2720
-Wire Bus Line
-	9605 1920 9605 2620
-Wire Bus Line
-	14845 5890 14845 6590
-Wire Bus Line
-	1175 3525 1175 4225
-Wire Bus Line
-	7165 5800 7165 6855
-Wire Bus Line
-	3870 2725 3870 4225
 $Comp
 L power:GND #PWR09
@@
 Text Label 9230 1320 0    50   ~ 0
 audio_out
+Connection ~ 11655 3015
+Wire Wire Line
+	11655 3015 10400 3015
+Wire Wire Line
+	12385 3015 11655 3015
+$Comp
+L Device:R_POT RV2
+U 1 1 64350FB5
+P 11805 3450
+F 0 "RV2" V 11598 3450 50  0000 C CNN
+F 1 "1M" V 11689 3450 50  0000 C CNN
+F 2 "ReSeed:Potentiometer_Vertical" H 11805 3450 50  0001 C CNN
+F 3 "~" H 11805 3450 50  0001 C CNN
+	1    11805 3450
+	0    -1   1    0
+$EndComp
+$Comp
+L Device:R R7
+U 1 1 6340C3F1
+P 11805 3885
+F 0 "R7" H 11735 3839 50  0000 R CNN
+F 1 "180k" H 11735 3930 50  0000 R CNN
+F 2 "Resistor_THT:R_Axial_DIN0207_L6.3mm_D2.5mm_P10.16mm_Horizontal" V 11735 3885 50  0001 C CNN
+F 3 "~" H 11805 3885 50  0001 C CNN
+	1    11805 3885
+	-1   0    0    1
+$EndComp
+$Comp
+L power:GND #PWR016
+U 1 1 6340CB1D
+P 11805 4110
+F 0 "#PWR016" H 11805 3860 50  0001 C CNN
+F 1 "GND" H 11810 3937 50  0000 C CNN
+F 2 "" H 11805 4110 50  0001 C CNN
+F 3 "" H 11805 4110 50  0001 C CNN
+	1    11805 4110
+	1    0    0    -1
+$EndComp
+Wire Wire Line
+	11805 4035 11805 4110
+Wire Wire Line
+	11655 3015 11655 3350
+$Comp
+L Connector:Conn_01x03_Male SW1
+U 1 1 6436DD9D
+P 11295 3350
+F 0 "SW1" H 11403 3631 50  0000 C CNN
+F 1 "SW_DIGIFIX" H 11403 3540 50  0000 C CNN
+F 2 "Connector_PinHeader_2.54mm:PinHeader_1x03_P2.54mm_Vertical" H 11295 3350 50  0001 C CNN
+F 3 "~" H 11295 3350 50  0001 C CNN
+	1    11295 3350
+	1    0    0    -1
+$EndComp
+Wire Wire Line
+	11495 3350 11655 3350
+Wire Wire Line
+	11495 3450 11655 3450
+NoConn ~ 11495 3250
+Wire Wire Line
+	11805 3600 11805 3735
+NoConn ~ 11955 3450
+Wire Bus Line
+	9365 5800 9365 6055
+Wire Bus Line
+	7120 2320 7120 2720
+Wire Bus Line
+	9605 1920 9605 2620
+Wire Bus Line
+	14845 5890 14845 6590
+Wire Bus Line
+	1175 3525 1175 4225
+Wire Bus Line
+	7165 5800 7165 6855
+Wire Bus Line
+	3870 2725 3870 4225
 $EndSCHEMATC
