File: ReSeed.sch (KiCad schematic (older format))
At the start: 47 parts, among them CN1 EDGE_CONNECTOR, CN2 AUDIO_OUT, CN3 AUDIO_IN, CN4 DB9_MALE, Q1 BC547C, SW1 SW_DIGIFIX, U1 MOS_8580, U2 CD4520BE, U3 74LS245, U4 GAL16V8, U5 TL497ACN

Commit message: Add P/Ns
Parts:
- C6: MouserPN (none) -> 810-FG28C0G1H471JNT6
- C7: MouserPN (none) -> 810-FG28X7R1H104KNT0
- CN2, CN3: MouserPN (none) -> 490-SJ1-3525N
- JP1, V0, V1: MouserPN (none) -> ---
- Q1: MouserPN (none) -> 512-BC549CTA
- R1, R2: MouserPN (none) -> 660-MF1/4LCT52R101G
- R3, R5: MouserPN (none) -> 603-MFR-25FBF52-1K
- R4: MouserPN (none) -> 603-MFR-25FTF52-10K
- R6: MouserPN (none) -> 603-MF0207FTE52-180K
- R7: MouserPN (none) -> 603-MFR-25FBF52-100K
- R8: MouserPN 603-MF0207FRE52-1R -> 603-MFR50SFTE52-3R3
- RV1: MouserPN (none) -> 652-3306P-1-103
- RV2: MouserPN (none) -> 652-3306P-1-105
- U2: MouserPN 595-CD74HCT4520E -> 595-CD4520BE
- U3: MouserPN 595-SN74HCT245N -> 595-SN74HCT245N
- U4: MouserPN 556-AF16V8B15PU -> 556-AF16V8B15PU
- U5: MouserPN 595-TL497ACNE4 -> 595-TL497ACNE4
Changed lines of the file:
@@
 F 2 "Package_DIP:DIP-16_W7.62mm_Socket_LongPads" H 5915 2220 50  0001 C CNN
 F 3 "http://www.intersil.com/content/dam/Intersil/documents/cd45/cd4518bms-20bms.pdf" H 5915 2220 50  0001 C CNN
-F 4 "595-CD74HCT4520E" H 5915 2220 50  0001 C CNN "MouserPN"
+F 4 "595-CD4520BE" H 5915 2220 50  0001 C CNN "MouserPN"
 	1    5915 2220
 	1    0    0    -1
@@
 F 2 "Package_DIP:DIP-16_W7.62mm_Socket_LongPads" H 2615 8190 50  0001 C CNN
 F 3 "http://www.intersil.com/content/dam/Intersil/documents/cd45/cd4518bms-20bms.pdf" H 2615 8190 50  0001 C CNN
-F 4 "595-CD74HCT4520E" H 2615 8190 50  0001 C CNN "MouserPN"
+F 4 "595-CD4520BE" H 2615 8190 50  0001 C CNN "MouserPN"
 	2    2615 8190
 	1    0    0    -1
@@
 F 2 "Package_DIP:DIP-16_W7.62mm_Socket_LongPads" H 2885 9770 50  0001 C CNN
 F 3 "http://www.intersil.com/content/dam/Intersil/documents/cd45/cd4518bms-20bms.pdf" H 2885 9770 50  0001 C CNN
-F 4 "595-CD74HCT4520E" H 2885 9770 50  0001 C CNN "MouserPN"
+F 4 "595-CD4520BE" H 2885 9770 50  0001 C CNN "MouserPN"
 	3    2885 9770
 	1    0    0    -1
@@
 F 2 "Package_DIP:DIP-20_W7.62mm_Socket_LongPads" H 8265 6555 50  0001 C CNN
 F 3 "" H 8265 6555 50  0001 C CNN
-F 4 " 556-AF16V8B15PU" H 8265 6555 50  0001 C CNN "MouserPN"
+F 4 "556-AF16V8B15PU" H 8265 6555 50  0001 C CNN "MouserPN"
 	1    8265 6555
 	1    0    0    -1
@@
 F 2 "Package_DIP:DIP-14_W7.62mm_Socket_LongPads" H 8220 9515 50  0001 C CNN
 F 3 "http://www.ti.com/lit/ds/symlink/tl497a.pdf" H 8220 9515 50  0001 C CNN
-F 4 " 595-TL497ACNE4 " H 8220 9515 50  0001 C CNN "MouserPN"
+F 4 "595-TL497ACNE4 " H 8220 9515 50  0001 C CNN "MouserPN"
 	1    8220 9515
 	1    0    0    -1
@@
 F 2 "Package_DIP:DIP-20_W7.62mm_Socket_LongPads" H 13840 6490 50  0001 C CNN
 F 3 "http://www.ti.com/lit/gpn/sn74LS245" H 13840 6490 50  0001 C CNN
-F 4 " 595-SN74HCT245N" H 13840 6490 50  0001 C CNN "MouserPN"
+F 4 "595-SN74HCT245N" H 13840 6490 50  0001 C CNN "MouserPN"
 	1    13840 6490
 	1    0    0    -1
@@
 F 2 "Resistor_THT:R_Axial_DIN0207_L6.3mm_D2.5mm_P10.16mm_Horizontal" V 6860 9165 50  0001 C CNN
 F 3 "~" H 6930 9165 50  0001 C CNN
-F 4 "603-MF0207FRE52-1R" H 6930 9165 50  0001 C CNN "MouserPN"
+F 4 "603-MFR50SFTE52-3R3" H 6930 9165 50  0001 C CNN "MouserPN"
 	1    6930 9165
 	1    0    0    -1
@@
 F 2 "Resistor_THT:R_Axial_DIN0207_L6.3mm_D2.5mm_P10.16mm_Horizontal" V 9645 1720 50  0001 C CNN
 F 3 "~" H 9715 1720 50  0001 C CNN
+F 4 "660-MF1/4LCT52R101G" H 9715 1720 50  0001 C CNN "MouserPN"
 	1    9715 1720
 	0    1    1    0
@@
 F 2 "Resistor_THT:R_Axial_DIN0207_L6.3mm_D2.5mm_P10.16mm_Horizontal" V 9645 1620 50  0001 C CNN
 F 3 "~" H 9715 1620 50  0001 C CNN
+F 4 "660-MF1/4LCT52R101G" H 9715 1620 50  0001 C CNN "MouserPN"
 	1    9715 1620
 	0    1    1    0
@@
 F 2 "Resistor_THT:R_Axial_DIN0207_L6.3mm_D2.5mm_P10.16mm_Horizontal" V 11060 1320 50  0001 C CNN
 F 3 "~" H 11130 1320 50  0001 C CNN
+F 4 "603-MFR-25FTF52-10K" H 11130 1320 50  0001 C CNN "MouserPN"
 	1    11130 1320
 	0    1    1    0
@@
 F 2 "Package_TO_SOT_THT:TO-92_HandSolder" H 12640 1245 50  0001 L CIN
 F 3 "https://www.onsemi.com/pub/Collateral/BC550-D.pdf" H 12440 1320 50  0001 L CNN
+F 4 "512-BC549CTA" H 12440 1320 50  0001 C CNN "MouserPN"
 	1    12440 1320
 	1    0    0    -1
@@
 F 2 "Capacitor_THT:C_Disc_D7.0mm_W2.5mm_P5.00mm" H 12313 1475 50  0001 C CNN
 F 3 "~" H 12275 1625 50  0001 C CNN
+F 4 "810-FG28C0G1H471JNT6" H 12275 1625 50  0001 C CNN "MouserPN"
 	1    12275 1625
 	0    1    1    0
@@
 F 2 "Resistor_THT:R_Axial_DIN0207_L6.3mm_D2.5mm_P10.16mm_Horizontal" V 12470 1905 50  0001 C CNN
 F 3 "~" H 12540 1905 50  0001 C CNN
+F 4 "603-MFR-25FBF52-1K" H 12540 1905 50  0001 C CNN "MouserPN"
 	1    12540 1905
 	-1   0    0    1
@@
 F 2 "ReSeed:Pot_Bourns_3306P" H 13420 1905 50  0001 C CNN
 F 3 "~" H 13420 1905 50  0001 C CNN
+F 4 "652-3306P-1-103" H 13420 1905 50  0001 C CNN "MouserPN"
 	1    13420 1905
 	1    0    0    -1
@@
 F 2 "Resistor_THT:R_Axial_DIN0207_L6.3mm_D2.5mm_P10.16mm_Horizontal" V 13445 3295 50  0001 C CNN
 F 3 "~" H 13515 3295 50  0001 C CNN
+F 4 "603-MFR-25FBF52-100K" H 13515 3295 50  0001 C CNN "MouserPN"
 	1    13515 3295
 	-1   0    0    1
@@
 F 2 "ReSeed:AudioJack_SJ1-3525N" H 14965 3215 50  0001 C CNN
 F 3 "~" H 14965 3215 50  0001 C CNN
+F 4 "490-SJ1-3525N" H 14965 3215 50  0001 C CNN "MouserPN"
 	1    14965 3215
 	-1   0    0    1
@@
 F 2 "ReSeed:Logo" H 15465 9505 50  0001 C CNN
 F 3 "" H 15465 9505 50  0001 C CNN
+F 4 "---" H 15465 9505 50  0001 C CNN "MouserPN"
 	1    15465 9505
 	1    0    0    -1
@@
 F 2 "ReSeed:cc_by_nc_sa" H 15465 9740 50  0001 C CNN
 F 3 "" H 15465 9740 50  0001 C CNN
+F 4 "---" H 15465 9740 50  0001 C CNN "MouserPN"
 	1    15465 9740
 	1    0    0    -1
@@
 F 2 "ReSeed:AudioJack_SJ1-3525N" H 14965 1845 50  0001 C CNN
 F 3 "~" H 14965 1845 50  0001 C CNN
+F 4 "490-SJ1-3525N" H 14965 1845 50  0001 C CNN "MouserPN"
 	1    14965 1845
 	-1   0    0    1
@@
 F 2 "Resistor_THT:R_Axial_DIN0207_L6.3mm_D2.5mm_P10.16mm_Horizontal" V 10635 1600 50  0001 C CNN
 F 3 "~" H 10705 1600 50  0001 C CNN
+F 4 "603-MFR-25FBF52-1K" H 10705 1600 50  0001 C CNN "MouserPN"
 	1    10705 1600
 	-1   0    0    1
@@
 F 2 "Capacitor_THT:C_Disc_D7.0mm_W2.5mm_P5.00mm" H 13068 790 50  0001 C CNN
 F 3 "~" H 13030 940 50  0001 C CNN
+F 4 "810-FG28X7R1H104KNT0" H 13030 940 50  0001 C CNN "MouserPN"
 	1    13030 940
 	0    1    1    0
@@
 F 2 "ReSeed:Pot_Bourns_3306P" H 11805 3450 50  0001 C CNN
 F 3 "~" H 11805 3450 50  0001 C CNN
+F 4 "652-3306P-1-105" H 11805 3450 50  0001 C CNN "MouserPN"
 	1    11805 3450
 	0    -1   1    0
@@
 F 2 "Resistor_THT:R_Axial_DIN0207_L6.3mm_D2.5mm_P10.16mm_Horizontal" V 11735 3885 50  0001 C CNN
 F 3 "~" H 11805 3885 50  0001 C CNN
+F 4 "603-MF0207FTE52-180K" H 11805 3885 50  0001 C CNN "MouserPN"
 	1    11805 3885
 	-1   0    0    1
@@
 F 2 "Jumper:SolderJumper-2_P1.3mm_Bridged_RoundedPad1.0x1.5mm" H 14550 2915 50  0001 C CNN
 F 3 "~" H 14550 2915 50  0001 C CNN
+F 4 "---" H 14550 2915 50  0001 C CNN "MouserPN"
 	1    14550 2915
 	1    0    0    -1
