File: ReSeed.sch (KiCad schematic (older format))
At the start: 59 parts, among them CN1 EDGE_CONNECTOR, CN2 AUDIO_OUT, CN3 AUDIO_IN, CN4 DB9_MALE, Q1 BC549C, Q101 2SC1815, SW1 SW_DIGIFIX, U1 MOS_8580, U105 STEPUP_MT3608, U2 CD74HCT4520E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

Commit message: Ready for 44-pin version
Parts:
- removed CN1: EDGE_CONNECTOR, ReSeed:C16_Cart_Conn, symbol C16-Exp-Port:C16-Exp-Port
- added CN1: EDGE_CONNECTOR, ReSeed:C16-Exp-Port-44Pin, symbol C16-Exp-Port-44Pin:C16_EXP_PORT_44PIN
Connections:
- net GND: now also CN1.1 (GND), CN1.22 (GND), CN1.A (GND), CN1.Z (GND)
- net a0: now also CN1.Y (A0)
- net a1: now also CN1.X (A1)
- net a10: now also CN1.M (A10)
- net a11: now also CN1.L (A11)
- net a12: now also CN1.K (A12)
- net a13: now also CN1.J (A13)
- net a14: now also CN1.H (A14)
- net a15: now also CN1.F (A15)
- net a2: now also CN1.W (A2)
- net a3: now also CN1.V (A3)
- net a4: now also CN1.U (A4)
- net a5: now also CN1.T (A5)
- net a6: now also CN1.S (A6)
- net a7: now also CN1.R (A7)
- net a8: now also CN1.P (A8)
- net a9: now also CN1.N (A9)
- net d0: now also CN1.21 (D0)
- net d1: now also CN1.20 (D1)
- net d2: now also CN1.19 (D2)
- net d3: now also CN1.18 (D3)
- net d4: now also CN1.17 (D4)
- net d5: now also CN1.16 (D5)
- net d6: now also CN1.15 (D6)
- net d7: now also CN1.14 (D7)
- net ext_audio: now also CN1.9 (EXT_AUDIO)
- net mux: now also CN1.13 (MUX)
- net phi2: now also CN1.6 (PHI2)
- net r_~w: now also CN1.5 (R/~W)
- net ~reset: now also CN1.C (~RESET)
- net at FB1.1: now also CN1.2 (+5V), CN1.3 (+5V)
- no-connect marks 26 -> 23
Changed lines of the file:
@@
 Sheet 1 1
 Title "ReSeed"
-Date "2023-02-09"
+Date "2023-10-04"
 Rev "2git"
 Comp "SukkoPera/Kinmami"
@@
 L power:GND #PWR021
 U 1 1 62087AD2
-P 2250 3895
-F 0 "#PWR021" H 2250 3645 50  0001 C CNN
-F 1 "GND" H 2255 3722 50  0000 C CNN
-F 2 "" H 2250 3895 50  0001 C CNN
-F 3 "" H 2250 3895 50  0001 C CNN
-	1    2250 3895
+P 2250 3595
+F 0 "#PWR021" H 2250 3345 50  0001 C CNN
+F 1 "GND" H 2255 3422 50  0000 C CNN
+F 2 "" H 2250 3595 50  0001 C CNN
+F 3 "" H 2250 3595 50  0001 C CNN
+	1    2250 3595
 	1    0    0    -1
 $EndComp
@@
 ANALOG PADDLE/JOYSTICK PORT
 $Comp
-L C16-Exp-Port:C16-Exp-Port CN1
-U 1 1 62403A40
-P 3140 2500
-F 0 "CN1" H 3140 4065 50  0000 C CNN
-F 1 "EDGE_CONNECTOR" H 3140 3974 50  0000 C CNN
-F 2 "ReSeed:C16_Cart_Conn" H 3140 850 50  0001 C CNN
-F 3 "DOCUMENTATION" H 3140 750 50  0001 C CNN
-F 4 "---" H 3140 2500 50  0001 C CNN "MouserPN"
-F 5 "EDGE_CONNECTOR" H 3140 2500 50  0001 C CNN "Value"
-	1    3140 2500
-	1    0    0    -1
-$EndComp
-$Comp
 L power:GND #PWR022
 U 1 1 62418CFF
-P 4030 3895
-F 0 "#PWR022" H 4030 3645 50  0001 C CNN
-F 1 "GND" H 4035 3722 50  0000 C CNN
-F 2 "" H 4030 3895 50  0001 C CNN
-F 3 "" H 4030 3895 50  0001 C CNN
-	1    4030 3895
+P 4030 3595
+F 0 "#PWR022" H 4030 3345 50  0001 C CNN
+F 1 "GND" H 4035 3422 50  0000 C CNN
+F 2 "" H 4030 3595 50  0001 C CNN
+F 3 "" H 4030 3595 50  0001 C CNN
+	1    4030 3595
 	-1   0    0    -1
 $EndComp
-NoConn ~ 2390 1800
 NoConn ~ 2390 1900
 NoConn ~ 2390 2000
-NoConn ~ 2390 2100
 NoConn ~ 2390 2200
 NoConn ~ 2390 2300
-NoConn ~ 2390 2500
-NoConn ~ 2390 3400
 NoConn ~ 3890 1400
 NoConn ~ 3890 1600
@@
 Text Label 1785 1700 0    50   ~ 0
 r_~w
-Text Label 1785 2400 0    50   ~ 0
+Text Label 1785 2500 0    50   ~ 0
 mux
 Entry Wire Line
@@
 Text Label 4280 3300 2    50   ~ 0
 a0
-Text Label 1785 3500 0    50   ~ 0
+Text Label 1785 2100 0    50   ~ 0
 ext_audio
 $Comp
@@
 	1    0    0    -1
 $EndComp
-Text Label 1785 3600 0    50   ~ 0
+Text Label 1785 1800 0    50   ~ 0
 phi2
 $Comp
@@
 reset
 Wire Wire Line
-	2390 3700 2250 3700
-Connection ~ 2250 3700
-Wire Wire Line
-	2250 3700 2250 3895
+	2390 3400 2250 3400
+Connection ~ 2250 3400
+Wire Wire Line
+	2250 3400 2250 3595
 Wire Wire Line
 	2390 1500 2140 1500
@@
 	2250 1300 2390 1300
 Wire Wire Line
-	3890 3700 4030 3700
-Connection ~ 4030 3700
-Wire Wire Line
-	4030 3700 4030 3895
+	3890 3400 4030 3400
+Connection ~ 4030 3400
+Wire Wire Line
+	4030 3400 4030 3595
 Wire Wire Line
 	4030 1300 3890 1300
 Wire Wire Line
-	4030 1300 4030 3700
-Wire Wire Line
-	2250 1300 2250 3700
+	4030 1300 4030 3400
+Wire Wire Line
+	2250 1300 2250 3400
 Wire Wire Line
 	2390 1400 2140 1400
@@
 	2390 1700 1785 1700
 Wire Wire Line
-	2390 2400 1785 2400
+	2390 2500 1785 2500
 Wire Wire Line
 	2390 2600 1785 2600
@@
 	1685 2500 1255 2500
 Wire Wire Line
-	2390 3500 1785 3500
-Wire Wire Line
-	2390 3600 1785 3600
+	2390 2100 1785 2100
+Wire Wire Line
+	2390 1800 1785 1800
 Wire Wire Line
 	1320 10315 1320 10410
@@
 Wire Notes Line
 	9495 2025 9495 1030
+$Comp
+L C16-Exp-Port-44Pin:C16_EXP_PORT_44PIN CN1
+U 1 1 65200D43
+P 3140 2350
+F 0 "CN1" H 3140 3765 50  0000 C CNN
+F 1 "EDGE_CONNECTOR" H 3140 3674 50  0000 C CNN
+F 2 "ReSeed:C16-Exp-Port-44Pin" H 3140 900 50  0001 C CNN
+F 3 "" H 3140 800 50  0001 C CNN
+	1    3140 2350
+	1    0    0    -1
+$EndComp
+NoConn ~ 2390 2400
 Wire Bus Line
 	8650 5890 8650 6745
